File: Placa V2.0/v2.1/placa1.brd (EAGLE design)
At the start: 69.5 x 40 mm, 8 parts, among them IC1 LD117AS50TR

Commit message: Super actualización
Parts:
- removed R: 4K7, rcl:R1206
- removed U1: (no value), RHT03_DHT-22_AM2302:RHT03_DHT-22/RA
- added U$1: (no value), DHT11:DHT11
- moved ESP8266 42.4 mm to (16.5, 27.9), turned to 270 degrees
- moved JP1 35.3 mm to (19.1, 18.4), turned to 180 degrees
- moved IC1 25.4 mm to (19.1, 12.1), turned to 0 degrees
- moved C1 25.3 mm to (13.3, 8.89), turned to 0 degrees
- moved OLED 17.3 mm to (15.9, 37.5)
- moved C2 11.8 mm to (24.4, 7.97), turned to 90 degrees
Connections:
- net SCL renamed N$3
- new net N$4: ESP8266.RX, JP1.3
- net 3V3: now also U$1.VCC; no longer R.1, U1.VDD
- net 5V: now also JP1.5
- net DATA: now also U$1.DATA; no longer R.2, U1.DATA
- net GND: now also JP1.1, U$1.GND; no longer U1.GND
Routing:
- net GND: track 0.00 -> 70.2 mm
- net DATA: track 74.2 -> 19.7 mm
- net 3V3: track 126.5 -> 75.2 mm, vias 1 -> 0
- net N$3: track 33.0 -> 15.9 mm
- net N$4: track 0.00 -> 13.0 mm
- net SDA: track 24.1 -> 20.1 mm
- net 5V: track 10.7 -> 12.0 mm
- removed copper zone on layer 16, net GND
Other:
- board size 69.5 x 40 mm -> 33 x 54 mm
