File: Placa V2.0/placa1.sch (EAGLE design)
At the start: 7 parts, among them IC1 LD117AS50TR

Commit message: cambios en placa
Parts:
- removed U$1: (no value), DHT11:DHT11
- added J1: STEREOJACKSJ1-352XNG, Ai_Connectors:STEREOJACKSJ1-352XNG
- added U1: (no value), dht22:RHT03_DHT-22_AM2302RA
Connections:
- removed net N$4: ESP8266.RXD, JP1.3
- new net RX: ESP8266.RXD, J1.RNG, J1.RSH
- net 3V3: now also J1.TIP, J1.TSH, U1.VDD; no longer U$1.VCC
- net DATA: now also U1.DATA; no longer U$1.DATA
- net GND: now also J1.GND, U1.GND; no longer U$1.GND
Changed lines of the file:
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@@
 <layer number="115" name="ReferenceISLANDS" color="7" fill="1" visible="yes" active="yes"/>
 <layer number="116" name="Patch_BOT" color="9" fill="4" visible="yes" active="yes"/>
+<layer number="117" name="mPads" color="7" fill="1" visible="no" active="no"/>
 <layer number="118" name="Rect_Pads" color="7" fill="1" visible="yes" active="yes"/>
+<layer number="119" name="mUnrouted" color="7" fill="1" visible="no" active="no"/>
+<layer number="120" name="mDimension" color="7" fill="1" visible="no" active="no"/>
 <layer number="121" name="_tsilk" color="7" fill="1" visible="yes" active="yes"/>
 <layer number="122" name="_bsilk" color="7" fill="1" visible="yes" active="yes"/>
@@
 <layer number="128" name="_bValues" color="7" fill="1" visible="yes" active="yes"/>
 <layer number="129" name="Mask" color="7" fill="1" visible="yes" active="yes"/>
+<layer number="130" name="mbStop" color="7" fill="1" visible="no" active="no"/>
 <layer number="131" name="tAdjust" color="7" fill="1" visible="yes" active="yes"/>
 <layer number="132" name="bAdjust" color="7" fill="1" visible="yes" active="yes"/>
+<layer number="133" name="mtFinish" color="7" fill="1" visible="no" active="no"/>
+<layer number="134" name="mbFinish" color="7" fill="1" visible="no" active="no"/>
+<layer number="135" name="mtGlue" color="7" fill="1" visible="no" active="no"/>
+<layer number="136" name="mbGlue" color="7" fill="1" visible="no" active="no"/>
+<layer number="137" name="mtTest" color="7" fill="1" visible="no" active="no"/>
+<layer number="138" name="mbTest" color="7" fill="1" visible="no" active="no"/>
+<layer number="139" name="mtKeepout" color="7" fill="1" visible="no" active="no"/>
+<layer number="140" name="mbKeepout" color="7" fill="1" visible="no" active="no"/>
+<layer number="141" name="mtRestrict" color="7" fill="1" visible="no" active="no"/>
+<layer number="142" name="mbRestrict" color="7" fill="1" visible="no" active="no"/>
+<layer number="143" name="mvRestrict" color="7" fill="1" visible="no" active="no"/>
 <layer number="144" name="Drill_legend" color="7" fill="1" visible="yes" active="yes"/>
+<layer number="145" name="mHoles" color="7" fill="1" visible="no" active="no"/>
+<layer number="146" name="mMilling" color="7" fill="1" visible="no" active="no"/>
+<layer number="147" name="mMeasures" color="7" fill="1" visible="no" active="no"/>
+<layer number="148" name="mDocument" color="7" fill="1" visible="no" active="no"/>
+<layer number="149" name="mReference" color="7" fill="1" visible="no" active="no"/>
 <layer number="150" name="Notes" color="7" fill="1" visible="yes" active="yes"/>
 <layer number="151" name="HeatSink" color="7" fill="1" visible="yes" active="yes"/>
@@
 <layer number="154" name="FabDoc2" color="7" fill="1" visible="yes" active="yes"/>
 <layer number="155" name="FabDoc3" color="7" fill="1" visible="yes" active="yes"/>
+<layer number="191" name="mNets" color="7" fill="1" visible="no" active="no"/>
+<layer number="192" name="mBusses" color="7" fill="1" visible="no" active="no"/>
+<layer number="193" name="mPins" color="7" fill="1" visible="no" active="no"/>
+<layer number="194" name="mSymbols" color="7" fill="1" visible="no" active="no"/>
+<layer number="195" name="mNames" color="7" fill="1" visible="no" active="no"/>
+<layer number="196" name="mValues" color="7" fill="1" visible="no" active="no"/>
 <layer number="199" name="Contour" color="7" fill="1" visible="yes" active="yes"/>
 <layer number="200" name="200bmp" color="1" fill="10" visible="yes" active="yes"/>
@@
 <part name="GND5" library="supply1" deviceset="GNDA" device=""/>
 <part name="GND2" library="supply1" deviceset="GNDA" device=""/>
-<part name="U$1" library="DHT11" deviceset="DHT11" device=""/>
 <part name="JP1" library="pinhead" library_urn="urn:adsk.eagle:library:325" deviceset="PINHD-1X5" device=""/>
+<part name="J1" library="Ai_Connectors" deviceset="STEREOJACK" device="SJ1-352XNG"/>
+<part name="GND1" library="supply1" deviceset="GNDA" device=""/>
+<part name="U1" library="dht22" deviceset="RHT03_DHT-22_AM2302" device="RA"/>
 </parts>
 <sheets>
@@
 <instance part="GND5" gate="1" x="91.44" y="53.34" smashed="yes"/>
 <instance part="GND2" gate="1" x="86.36" y="40.64" smashed="yes"/>
-<instance part="U$1" gate="G$1" x="106.68" y="30.48" rot="MR90"/>
 <instance part="JP1" gate="A" x="0" y="55.88" rot="R180"/>
+<instance part="J1" gate="G$1" x="109.22" y="15.24" rot="R180"/>
+<instance part="GND1" gate="1" x="93.98" y="7.62" smashed="yes"/>
+<instance part="U1" gate="G$1" x="104.14" y="35.56" rot="MR180"/>
 </instances>
 <busses>
@@
 <junction x="45.72" y="55.88"/>
 <wire x1="45.72" y1="27.94" x2="93.98" y2="27.94" width="0.1524" layer="91"/>
-<pinref part="U$1" gate="G$1" pin="VCC"/>
+<pinref part="U1" gate="G$1" pin="VDD"/>
 </segment>
 <segment>
@@
 <label x="88.9" y="50.8" size="1.27" layer="95" rot="R180" xref="yes"/>
 </segment>
+<segment>
+<pinref part="J1" gate="G$1" pin="TIP"/>
+<wire x1="100.33" y1="20.32" x2="96.52" y2="20.32" width="0.1524" layer="91"/>
+<pinref part="J1" gate="G$1" pin="TSH"/>
+<wire x1="100.33" y1="17.78" x2="96.52" y2="17.78" width="0.1524" layer="91"/>
+<wire x1="96.52" y1="17.78" x2="96.52" y2="20.32" width="0.1524" layer="91"/>
+<wire x1="96.52" y1="20.32" x2="93.98" y2="20.32" width="0.1524" layer="91"/>
+<junction x="96.52" y="20.32"/>
+<label x="93.98" y="20.32" size="1.27" layer="95" rot="R180" xref="yes"/>
+</segment>
 </net>
 <net name="DATA" class="0">
 <segment>
-<wire x1="93.98" y1="30.48" x2="88.9" y2="30.48" width="0.1524" layer="91"/>
-<wire x1="88.9" y1="30.48" x2="88.9" y2="35.56" width="0.1524" layer="91"/>
 <pinref part="ESP8266" gate="G$1" pin="TXD"/>
 <wire x1="48.26" y1="53.34" x2="48.26" y2="35.56" width="0.1524" layer="91"/>
 <wire x1="48.26" y1="35.56" x2="88.9" y2="35.56" width="0.1524" layer="91"/>
-<pinref part="U$1" gate="G$1" pin="DATA"/>
+<pinref part="U1" gate="G$1" pin="DATA"/>
+<wire x1="93.98" y1="33.02" x2="88.9" y2="33.02" width="0.1524" layer="91"/>
+<wire x1="88.9" y1="33.02" x2="88.9" y2="35.56" width="0.1524" layer="91"/>
 </segment>
 </net>
@@
 </segment>
 <segment>
-<pinref part="U$1" gate="G$1" pin="GND"/>
-<wire x1="93.98" y1="35.56" x2="91.44" y2="35.56" width="0.1524" layer="91"/>
-<wire x1="91.44" y1="35.56" x2="91.44" y2="43.18" width="0.1524" layer="91"/>
+<pinref part="J1" gate="G$1" pin="GND"/>
+<pinref part="GND1" gate="1" pin="GNDA"/>
+<wire x1="100.33" y1="10.16" x2="93.98" y2="10.16" width="0.1524" layer="91"/>
+</segment>
+<segment>
+<pinref part="U1" gate="G$1" pin="GND"/>
 <pinref part="GND2" gate="1" pin="GNDA"/>
-<wire x1="91.44" y1="43.18" x2="86.36" y2="43.18" width="0.1524" layer="91"/>
+<wire x1="93.98" y1="43.18" x2="86.36" y2="43.18" width="0.1524" layer="91"/>
 </segment>
 </net>
@@
 </segment>
 </net>
-<net name="N$4" class="0">
-<segment>
-<pinref part="JP1" gate="A" pin="3"/>
-<wire x1="2.54" y1="55.88" x2="-5.08" y2="55.88" width="0.1524" layer="91"/>
-<wire x1="-5.08" y1="55.88" x2="-5.08" y2="68.58" width="0.1524" layer="91"/>
+<net name="RX" class="0">
+<segment>
 <pinref part="ESP8266" gate="G$1" pin="RXD"/>
 <wire x1="-5.08" y1="68.58" x2="81.28" y2="68.58" width="0.1524" layer="91"/>
 <wire x1="81.28" y1="68.58" x2="81.28" y2="60.96" width="0.1524" layer="91"/>
-</segment>
-</net>
+<wire x1="-5.08" y1="15.24" x2="-5.08" y2="68.58" width="0.1524" layer="91"/>
+<pinref part="J1" gate="G$1" pin="RSH"/>
+<wire x1="100.33" y1="15.24" x2="96.52" y2="15.24" width="0.1524" layer="91"/>
+<pinref part="J1" gate="G$1" pin="RNG"/>
+<wire x1="100.33" y1="12.7" x2="96.52" y2="12.7" width="0.1524" layer="91"/>
+<wire x1="96.52" y1="12.7" x2="96.52" y2="15.24" width="0.1524" layer="91"/>
+<wire x1="-5.08" y1="15.24" x2="96.52" y2="15.24" width="0.1524" layer="91"/>
+<junction x="96.52" y="15.24"/>
+</segment>
+</net>
